File: _autosave-macropadfr.kicad_pcb (KiCad board)
At the start: 2 copper layers, 24 parts, among them K1 KEYSW, K2 KEYSW, K3 KEYSW, K4 KEYSW

Commit message: messed with the crystal and some pcb stuff
Parts:
- removed Resonating_Clock1: crystal1, Crystal:Crystal_SMD_3225-4Pin_3.2x2.5mm_HandSoldering
- added clock1: crystal1_gnd24, Crystal:Crystal_SMD_Abracon_ABM8G-4Pin_3.2x2.5mm, B.Cu at (200.4, 104.1)
Connections:
- CCryst1 pad 2: +5V -> GND
- CCryst2 pad 2: +5V -> GND
- Cd1 pad 2: +5V -> GND
- Cd2 pad 2: +5V -> GND
- Cd3 pad 2: +5V -> GND
- Cd4 pad 2: +5V -> GND
- Cu1 pad 2: +5V -> GND
- processor1 pad 23: +5V -> GND
- processor1 pad 35: +5V -> GND
- processor1 pad 43: +5V -> GND
- reset_switch1 pad 1: +5V -> GND
