File: _autosave-macropadfr.kicad_pcb (KiCad board)
At the start: 2 copper layers, 66.7 x 38.3 mm, 28 parts, among them K1 KEYSW, K2 KEYSW, K3 KEYSW, K4 KEYSW

Commit message: bom and gerbers for final
Other:
- board text added: "JLCJLCJLCJLC"
