File: macropadfr.kicad_sch (KiCad schematic)
At the start: 24 parts, among them K1 KEYSW, K2 KEYSW, K3 KEYSW, K4 KEYSW

Commit message: messed with the crystal and some pcb stuff
Parts:
- removed Resonating_Clock1: crystal1, Crystal:Crystal_SMD_3225-4Pin_3.2x2.5mm_HandSoldering, symbol keyboard parts:XTAL_GND
- added clock1: crystal1_gnd24, Crystal:Crystal_SMD_Abracon_ABM8G-4Pin_3.2x2.5mm, symbol Device:Crystal_GND24
Connections:
- net +5V: no longer CCryst1.2, CCryst2.2, Cd1.2, Cd2.2, Cd3.2, Cd4.2, Cu1.2, processor1.23 (GND), processor1.35 (GND), processor1.43 (GND), reset_switch1.1
- net at CCryst2.1, processor1.17 (XTAL2): now also clock1.3
- net at CCryst1.1, processor1.16 (XTAL1): now also clock1.1
- new net GND: CCryst1.2, CCryst2.2, Cd1.2, Cd2.2, Cd3.2, Cd4.2, Cu1.2, clock1.2, clock1.4, processor1.23 (GND), processor1.35 (GND), processor1.43 (GND), reset_switch1.1

Commit message: deleted:    _autosave-macropadfr.kicad_pcb 	deleted:    macropadfr-backups/macropadfr-2022-02-24_200521.zip 	new file:   macropadfr-backups/macropadfr-2022-02-25_095033.zip 	new file:   macropadfr-backups/macropadfr-2022-02-25_095732.zip 	new file:   macropadfr-backups/macropadfr-2022-02-25_101325.zip 	new file:   macropadfr-backups/macropadfr-2022-02-25_102042.zip 	new file:   macropadfr-backups/macropadfr-2022-02-25_103804.zip 	new file:   macropadfr-backups/macropadfr-2022-02-25_104804.zip 	modified:   macropadfr.kicad_pcb 	modified:   macropadfr.kicad_prl 	modified:   macropadfr.kicad_pro 	modified:   macropadfr.kicad_sch 	modified:   macropadfr.net
Connections:
- net +5V is gone; now on net GND: Cusb1.1, Micro_USB1.5 (GND), Micro_USB1.6 (SHIELD), Rboot1.2, processor1.5 (UGnd)
- net GND: now also processor1.15 (GND)
- net VCC: now also processor1.14 (VCC)
- no-connect marks 26 -> 24
Changed lines of the file:
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@@
   (no_connect (at 55.88 99.06))
   (no_connect (at 55.88 96.52))
-  (no_connect (at 55.88 88.9))
-  (no_connect (at 55.88 86.36))
   (wire (pts (xy 135.89 73.66) (xy 138.43 73.66))
     (stroke (width 0) (type default) (color 0 0 0 0))
@@
     (stroke (width 0) (type default) (color 0 0 0 0))
   )
+  (wire (pts (xy 54.61 88.9) (xy 55.88 88.9))
+    (stroke (width 0) (type default) (color 0 0 0 0))
+  )
   (wire (pts (xy 114.3 76.2) (xy 116.84 76.2))
     (stroke (width 0) (type default) (color 0 0 0 0))
@@
     (stroke (width 0) (type default) (color 0 0 0 0))
   )
+  (wire (pts (xy 54.61 86.36) (xy 55.88 86.36))
+    (stroke (width 0) (type default) (color 0 0 0 0))
+  )
   (wire (pts (xy 110.49 53.34) (xy 111.76 53.34))
     (stroke (width 0) (type default) (color 0 0 0 0))
@@
   )
   (label "toD1" (at 138.43 63.5 90)
+    (effects (font (size 1.27 1.27)) (justify left bottom))
+  )
+  (label "UVCC" (at 49.53 55.88 0)
     (effects (font (size 1.27 1.27)) (justify left bottom))
   )
@@
   (symbol (lib_id "power:GND") (at 113.03 76.2 180) (unit 1)
     (in_bom yes) (on_board yes)
-    (property "Reference" "#PWR?" (id 0) (at 113.03 69.85 0)
+    (property "Reference" "#PWR0116" (id 0) (at 113.03 69.85 0)
       (effects (font (size 1.27 1.27)) hide)
     )
@@
   (symbol (lib_id "power:GND") (at 111.76 55.88 90) (unit 1)
     (in_bom yes) (on_board yes) (fields_autoplaced)
-    (property "Reference" "#PWR?" (id 0) (at 118.11 55.88 0)
+    (property "Reference" "#PWR0102" (id 0) (at 118.11 55.88 0)
       (effects (font (size 1.27 1.27)) hide)
     )
@@
   (symbol (lib_id "power:GND") (at 29.21 105.41 0) (unit 1)
     (in_bom yes) (on_board yes) (fields_autoplaced)
-    (property "Reference" "#PWR?" (id 0) (at 29.21 111.76 0)
+    (property "Reference" "#PWR0109" (id 0) (at 29.21 111.76 0)
       (effects (font (size 1.27 1.27)) hide)
     )
@@
   (symbol (lib_id "power:GND") (at 111.76 106.68 90) (unit 1)
     (in_bom yes) (on_board yes) (fields_autoplaced)
-    (property "Reference" "#PWR?" (id 0) (at 118.11 106.68 0)
+    (property "Reference" "#PWR0106" (id 0) (at 118.11 106.68 0)
       (effects (font (size 1.27 1.27)) hide)
     )
@@
     )
     (property "Datasheet" "" (id 3) (at 111.76 106.68 0)
+      (effects (font (size 1.27 1.27)) hide)
+    )
+    (pin "1")
+  )
+  (symbol (lib_id "power:GND") (at 40.64 63.5 270) (unit 1)
+    (in_bom yes) (on_board yes)
+    (property "Reference" "#PWR0104" (id 0) (at 34.29 63.5 0)
+      (effects (font (size 1.27 1.27)) hide)
+    )
+    (property "Value" "GND" (id 1) (at 33.02 63.5 90)
+      (effects (font (size 1.27 1.27)) (justify left))
+    )
+    (property "Footprint" "" (id 2) (at 40.64 63.5 0)
+      (effects (font (size 1.27 1.27)) hide)
+    )
+    (property "Datasheet" "" (id 3) (at 40.64 63.5 0)
       (effects (font (size 1.27 1.27)) hide)
     )
@@
     (pin "4")
   )
+  (symbol (lib_id "power:GND") (at 121.92 81.28 90) (unit 1)
+    (in_bom yes) (on_board yes)
+    (property "Reference" "#PWR0107" (id 0) (at 128.27 81.28 0)
+      (effects (font (size 1.27 1.27)) hide)
+    )
+    (property "Value" "GND" (id 1) (at 125.73 78.74 0)
+      (effects (font (size 1.27 1.27)) (justify right))
+    )
+    (property "Footprint" "" (id 2) (at 121.92 81.28 0)
+      (effects (font (size 1.27 1.27)) hide)
+    )
+    (property "Datasheet" "" (id 3) (at 121.92 81.28 0)
+      (effects (font (size 1.27 1.27)) hide)
+    )
+    (pin "1")
+  )
   (symbol (lib_id "power:GND") (at 21.59 80.01 270) (unit 1)
     (in_bom yes) (on_board yes)
-    (property "Reference" "#PWR?" (id 0) (at 15.24 80.01 0)
+    (property "Reference" "#PWR0112" (id 0) (at 15.24 80.01 0)
       (effects (font (size 1.27 1.27)) hide)
     )
@@
     (pin "1")
   )
-  (symbol (lib_id "keyboard parts:GND") (at 40.64 63.5 270) (unit 1)
-    (in_bom yes) (on_board yes)
-    (property "Reference" "#PWR0104" (id 0) (at 41.91 63.5 0)
-      (effects (font (size 0.508 0.508)) hide)
-    )
-    (property "Value" "GND" (id 1) (at 39.37 64.77 90)
-      (effects (font (size 0.762 0.762)) (justify left))
-    )
-    (property "Footprint" "" (id 2) (at 40.64 63.5 0)
-      (effects (font (size 1.524 1.524)))
-    )
-    (property "Datasheet" "" (id 3) (at 40.64 63.5 0)
-      (effects (font (size 1.524 1.524)))
-    )
-    (pin "1")
-  )
   (symbol (lib_id "Device:D") (at 160.02 68.58 90) (unit 1)
     (in_bom yes) (on_board yes) (fields_autoplaced)
@@
     (property "Datasheet" "" (id 3) (at 111.76 104.14 0)
       (effects (font (size 1.27 1.27)) hide)
-    )
-    (pin "1")
-  )
-  (symbol (lib_id "keyboard parts:GND") (at 121.92 81.28 90) (unit 1)
-    (in_bom yes) (on_board yes)
-    (property "Reference" "#PWR0107" (id 0) (at 120.65 81.28 0)
-      (effects (font (size 0.508 0.508)) hide)
-    )
-    (property "Value" "GND" (id 1) (at 123.19 82.55 90)
-      (effects (font (size 0.762 0.762)) (justify left))
-    )
-    (property "Footprint" "" (id 2) (at 121.92 81.28 0)
-      (effects (font (size 1.524 1.524)))
-    )
-    (property "Datasheet" "" (id 3) (at 121.92 81.28 0)
-      (effects (font (size 1.524 1.524)))
     )
     (pin "1")
@@
     (pin "6")
   )
+  (symbol (lib_id "power:VCC") (at 54.61 86.36 90) (unit 1)
+    (in_bom yes) (on_board yes) (fields_autoplaced)
+    (property "Reference" "#PWR0114" (id 0) (at 58.42 86.36 0)
+      (effects (font (size 1.27 1.27)) hide)
+    )
+    (property "Value" "VCC" (id 1) (at 50.8 86.3599 90)
+      (effects (font (size 1.27 1.27)) (justify left))
+    )
+    (property "Footprint" "" (id 2) (at 54.61 86.36 0)
+      (effects (font (size 1.27 1.27)) hide)
+    )
+    (property "Datasheet" "" (id 3) (at 54.61 86.36 0)
+      (effects (font (size 1.27 1.27)) hide)
+    )
+    (pin "1")
+  )
   (symbol (lib_id "keyboard parts:SW_PUSH") (at 29.21 82.55 0) (unit 1)
     (in_bom yes) (on_board yes)
@@
   (symbol (lib_id "power:GND") (at 25.4 134.62 0) (unit 1)
     (in_bom yes) (on_board yes) (fields_autoplaced)
-    (property "Reference" "#PWR?" (id 0) (at 25.4 140.97 0)
+    (property "Reference" "#PWR0111" (id 0) (at 25.4 140.97 0)
       (effects (font (size 1.27 1.27)) hide)
     )
@@
     )
     (property "Datasheet" "" (id 3) (at 25.4 134.62 0)
+      (effects (font (size 1.27 1.27)) hide)
+    )
+    (pin "1")
+  )
+  (symbol (lib_id "power:GND") (at 54.61 88.9 270) (unit 1)
+    (in_bom yes) (on_board yes) (fields_autoplaced)
+    (property "Reference" "#PWR0115" (id 0) (at 48.26 88.9 0)
+      (effects (font (size 1.27 1.27)) hide)
+    )
+    (property "Value" "GND" (id 1) (at 50.8 88.8999 90)
+      (effects (font (size 1.27 1.27)) (justify right))
+    )
+    (property "Footprint" "" (id 2) (at 54.61 88.9 0)
+      (effects (font (size 1.27 1.27)) hide)
+    )
+    (property "Datasheet" "" (id 3) (at 54.61 88.9 0)
       (effects (font (size 1.27 1.27)) hide)
     )
@@
       (reference "#PWR0101") (unit 1) (value "VCC") (footprint "")
     )
+    (path "/3fba7acf-fa87-44ee-bcba-0d2fba35b907"
+      (reference "#PWR0102") (unit 1) (value "GND") (footprint "")
+    )
     (path "/a5abddf4-c9da-4356-9d94-0797ffe079d4"
       (reference "#PWR0103") (unit 1) (value "VCC") (footprint "")
     )
-    (path "/abe7cdcf-4888-4549-a3a2-47acc5fadb69"
+    (path "/7d463918-3422-4690-9408-1c0c537d73d1"
       (reference "#PWR0104") (unit 1) (value "GND") (footprint "")
     )
@@
       (reference "#PWR0105") (unit 1) (value "VCC") (footprint "")
     )
-    (path "/c321a962-92c3-4854-85cc-a75fe8408312"
+    (path "/78f821b4-fa8b-45ba-b7ed-1755a5a99778"
+      (reference "#PWR0106") (unit 1) (value "GND") (footprint "")
+    )
+    (path "/8cce725f-d18d-406c-a0f7-7a76a7a13956"
       (reference "#PWR0107") (unit 1) (value "GND") (footprint "")
     )
@@
       (reference "#PWR0108") (unit 1) (value "VCC") (footprint "")
     )
+    (path "/70229269-a294-4022-a8d8-77b65c23a614"
+      (reference "#PWR0109") (unit 1) (value "GND") (footprint "")
+    )
     (path "/c62b3db5-3d87-46ac-bd18-de47d12485f1"
       (reference "#PWR0110") (unit 1) (value "VCC") (footprint "")
     )
+    (path "/f4c7f849-6d8f-4b6d-8594-94cf588648f9"
+      (reference "#PWR0111") (unit 1) (value "GND") (footprint "")
+    )
+    (path "/91616f55-534e-4b5a-9c3e-ffdff999b4cf"
+      (reference "#PWR0112") (unit 1) (value "GND") (footprint "")
+    )
     (path "/65dcec9d-388e-410b-90a8-70e55a181e1c"
       (reference "#PWR0113") (unit 1) (value "VCC") (footprint "")
     )
+    (path "/e011c297-361e-4d37-908e-0908c1ea3506"
+      (reference "#PWR0114") (unit 1) (value "VCC") (footprint "")
+    )
+    (path "/f5293239-4a66-4692-b786-f151687d6b79"
+      (reference "#PWR0115") (unit 1) (value "GND") (footprint "")
+    )
     (path "/2e792aef-05a3-4887-9c0d-c766b64075f1"
-      (reference "#PWR?") (unit 1) (value "GND") (footprint "")
-    )
-    (path "/3fba7acf-fa87-44ee-bcba-0d2fba35b907"
-      (reference "#PWR?") (unit 1) (value "GND") (footprint "")
-    )
-    (path "/70229269-a294-4022-a8d8-77b65c23a614"
-      (reference "#PWR?") (unit 1) (value "GND") (footprint "")
-    )
-    (path "/78f821b4-fa8b-45ba-b7ed-1755a5a99778"
-      (reference "#PWR?") (unit 1) (value "GND") (footprint "")
-    )
-    (path "/91616f55-534e-4b5a-9c3e-ffdff999b4cf"
-      (reference "#PWR?") (unit 1) (value "GND") (footprint "")
-    )
-    (path "/f4c7f849-6d8f-4b6d-8594-94cf588648f9"
-      (reference "#PWR?") (unit 1) (value "GND") (footprint "")
+      (reference "#PWR0116") (unit 1) (value "GND") (footprint "")
     )
     (path "/4da2e60c-eabc-45d7-8560-c8a1a496d984"

Commit message: rough draft done?
Connections:
- net toD2: now also D2.2 (A), K2.2; no longer D3.2 (A), K3.2
- net toD3: now also D3.2 (A), K3.2; no longer D2.2 (A), K2.2
Changed lines of the file:
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@@
     (effects (font (size 1.27 1.27)) (justify left bottom))
   )
-  (label "toD2" (at 160.02 63.5 90)
+  (label "toD3" (at 160.02 63.5 90)
     (effects (font (size 1.27 1.27)) (justify left bottom))
   )
@@
     (effects (font (size 1.27 1.27)) (justify left bottom))
   )
-  (label "toD3" (at 138.43 81.28 90)
+  (label "toD2" (at 138.43 81.28 90)
     (effects (font (size 1.27 1.27)) (justify left bottom))
   )
