File: macropadfr.kicad_pcb (KiCad board)
At the start: 2 copper layers, 24 parts, among them K1 KEYSW, K2 KEYSW, K3 KEYSW, K4 KEYSW

Commit message: deleted:    _autosave-macropadfr.kicad_pcb 	deleted:    macropadfr-backups/macropadfr-2022-02-24_200521.zip 	new file:   macropadfr-backups/macropadfr-2022-02-25_095033.zip 	new file:   macropadfr-backups/macropadfr-2022-02-25_095732.zip 	new file:   macropadfr-backups/macropadfr-2022-02-25_101325.zip 	new file:   macropadfr-backups/macropadfr-2022-02-25_102042.zip 	new file:   macropadfr-backups/macropadfr-2022-02-25_103804.zip 	new file:   macropadfr-backups/macropadfr-2022-02-25_104804.zip 	modified:   macropadfr.kicad_pcb 	modified:   macropadfr.kicad_prl 	modified:   macropadfr.kicad_pro 	modified:   macropadfr.kicad_sch 	modified:   macropadfr.net
Parts:
- removed Resonating_Clock1: crystal1, Crystal:Crystal_SMD_3225-4Pin_3.2x2.5mm_HandSoldering
- added clock1: crystal1_gnd24, Crystal:Crystal_SMD_Abracon_ABM8G-4Pin_3.2x2.5mm, B.Cu at (202.9, 103.8)
- moved Cu1 127.6 mm to (211.9, 88.1), turned to 0 degrees
- moved CCryst2 118.0 mm to (208.1, 104.8), turned to -90 degrees
- moved Cd4 117.4 mm to (204.8, 83.3), turned to -90 degrees
- moved reset_switch1 110.8 mm to (202.4, 76.2)
- moved Cd3 108.3 mm to (200.0, 83.3), turned to 90 degrees
- moved CCryst1 107.6 mm to (198.0, 104.8), turned to -90 degrees
- moved Rusb1 104.9 mm to (195.3, 81.0)
- moved Cd1 104.1 mm to (209.6, 100.0)
- moved Rusb2 100.0 mm to (195.3, 85.7)
- moved Rreset1 99.4 mm to (209.6, 83.3), turned to -90 degrees
- moved Cd2 94.7 mm to (195.3, 100.0), turned to 0 degrees
- moved Cusb1 94.1 mm to (211.9, 92.9)
- moved Rboot1 85.0 mm to (192.9, 92.9), turned to 90 degrees
- moved Micro_USB1 78.6 mm to (171.4, 76.2), turned to 0 degrees
- moved processor1 2.38 mm to (202.4, 92.9)
Connections:
- CCryst1 pad 2: +5V -> GND
- CCryst2 pad 2: +5V -> GND
- Cd1 pad 2: +5V -> GND
- Cd2 pad 2: +5V -> GND
- Cd3 pad 2: +5V -> GND
- Cd4 pad 2: +5V -> GND
- Cu1 pad 2: +5V -> GND
- Cusb1 pad 1: +5V -> GND
- Micro_USB1 pad 5: +5V -> GND
- Micro_USB1 pad 6: +5V -> GND
- Rboot1 pad 2: +5V -> GND
- processor1 pad 14: unconnected-(processor1-Pad14) -> VCC
- processor1 pad 15: unconnected-(processor1-Pad15) -> GND
- processor1 pad 23: +5V -> GND
- processor1 pad 35: +5V -> GND
- processor1 pad 43: +5V -> GND
- processor1 pad 5: +5V -> GND
- reset_switch1 pad 1: +5V -> GND

Commit message: rough draft done?
Parts:
- locked: renamed from Cu1; value 4.7u -> locked
- moved reset_switch1 31.1 mm to (204.0, 107.3), turned to 0 degrees
- moved CCryst1 25.8 mm to (198.7, 79.0), turned to 90 degrees
- moved CCryst2 25.8 mm to (207.9, 79.0), turned to 90 degrees
- moved clock1 24.0 mm to (203.4, 79.7), turned to 40 degrees
- moved Cd2 22.9 mm to (211.1, 83.5)
- moved Rreset1 22.5 mm to (196.2, 101.5)
- moved Cd1 20.8 mm to (196.9, 83.5)
- moved Rboot1 19.5 mm to (211.7, 98.2), turned to -90 degrees
- moved Cusb1 19.1 mm to (193.0, 90.2), turned to 0 degrees
- moved locked 18.9 mm to (194.5, 95.4), turned to 180 degrees
- moved Cd3 18.0 mm to (206.4, 100.2), turned to -90 degrees
- moved Cd4 17.1 mm to (201.6, 100.2)
- moved Rusb2 6.71 mm to (192.8, 79.5), turned to 0 degrees
- moved Rusb1 4.14 mm to (192.8, 84.2), turned to 0 degrees
- moved Micro_USB1 3.05 mm to (171.4, 79.2)
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Routing:
- net VCC: track 0.00 -> 90.5 mm
- net /col0: track 0.00 -> 75.8 mm, vias 0 -> 2
- net /col1: track 0.00 -> 57.4 mm, vias 0 -> 1
- net /row1: track 0.00 -> 44.5 mm
- net /row0: track 0.00 -> 43.7 mm, vias 0 -> 2
- net Net-(Rreset1-Pad2): track 0.00 -> 35.2 mm, vias 0 -> 2
- net Net-(Micro_USB1-Pad3): track 0.00 -> 27.9 mm
- net Net-(Micro_USB1-Pad2): track 0.00 -> 27.1 mm
- net Net-(Rusb2-Pad2): track 0.00 -> 15.1 mm
- net /toD4: track 0.00 -> 14.6 mm
- net /toD2: track 0.00 -> 13.7 mm
- net /toD1: track 0.00 -> 13.7 mm
- net /toD3: track 0.00 -> 13.7 mm
- net Net-(Rusb1-Pad2): track 0.00 -> 13.0 mm
- net Net-(CCryst1-Pad1): track 0.00 -> 9.55 mm
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- added copper zone on B.Cu, net GND
- added copper zone on F.Cu, net GND
Other:
- board outline added: 61.9 x 38.3 mm

Commit message: fixed some problems with connections
Routing:
- net GND: track 0.00 -> 51.3 mm, vias 0 -> 6
Changed lines of the file:
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@@
   (segment (start 197 90.25) (end 197.38125 90.63125) (width 0.25) (layer "B.Cu") (net 18))
   (segment (start 197.38125 90.63125) (end 198.3375 90.63125) (width 0.25) (layer "B.Cu") (net 18))
+  (segment (start 203.2 84.377856) (end 203.2 84.96875) (width 0.25) (layer "B.Cu") (net 25))
+  (segment (start 201.520366 82.698222) (end 203.2 84.377856) (width 0.25) (layer "B.Cu") (net 25))
+  (segment (start 198.907821 79.785929) (end 198.65625 80.0375) (width 0.25) (layer "B.Cu") (net 25))
   (segment (start 201.520366 80.282795) (end 201.520366 82.698222) (width 0.25) (layer "B.Cu") (net 25))
-  (segment (start 198.65625 80.0375) (end 198.907821 79.785929) (width 0.25) (layer "B.Cu") (net 25))
+  (segment (start 202.017232 79.785929) (end 198.907821 79.785929) (width 0.25) (layer "B.Cu") (net 25))
   (segment (start 202.017232 79.785929) (end 201.520366 80.282795) (width 0.25) (layer "B.Cu") (net 25))
-  (segment (start 203.2 84.377856) (end 203.2 84.96875) (width 0.25) (layer "B.Cu") (net 25))
-  (segment (start 198.907821 79.785929) (end 202.017232 79.785929) (width 0.25) (layer "B.Cu") (net 25))
-  (segment (start 201.520366 82.698222) (end 203.2 84.377856) (width 0.25) (layer "B.Cu") (net 25))
   (segment (start 207.90625 80.0375) (end 207.542821 79.674071) (width 0.25) (layer "B.Cu") (net 26))
   (segment (start 207.542821 79.674071) (end 204.795268 79.674071) (width 0.25) (layer "B.Cu") (net 26))
@@
   (segment (start 204.795268 79.674071) (end 204.795268 83.582588) (width 0.25) (layer "B.Cu") (net 26))
   (segment (start 204.795268 83.582588) (end 204 84.377856) (width 0.25) (layer "B.Cu") (net 26))
+  (segment (start 193.286053 92.173947) (end 193.226052 92.173947) (width 0.25) (layer "F.Cu") (net 43))
+  (segment (start 206.22 88.078356) (end 206.52 87.778356) (width 0.25) (layer "F.Cu") (net 43))
+  (segment (start 200.595735 91.425735) (end 200.595735 91.525735) (width 0.25) (layer "F.Cu") (net 43))
+  (segment (start 206.22 89.29) (end 206.22 88.078356) (width 0.25) (layer "F.Cu") (net 43))
+  (segment (start 193.226052 92.173947) (end 192.231454 93.168545) (width 0.25) (layer "F.Cu") (net 43))
+  (segment (start 200.595735 91.525735) (end 201.570333 92.500333) (width 0.25) (layer "F.Cu") (net 43))
+  (via (at 193.286053 92.173947) (size 0.8) (drill 0.4) (layers "F.Cu" "B.Cu") (net 43))
+  (via (at 201.570333 92.500333) (size 0.8) (drill 0.4) (layers "F.Cu" "B.Cu") (net 43))
+  (via (at 192.231454 93.168545) (size 0.8) (drill 0.4) (layers "F.Cu" "B.Cu") (net 43))
+  (via (at 206.22 89.29) (size 0.8) (drill 0.4) (layers "F.Cu" "B.Cu") (net 43))
+  (via (at 206.52 87.778356) (size 0.8) (drill 0.4) (layers "F.Cu" "B.Cu") (net 43))
+  (via (at 200.595735 91.425735) (size 0.8) (drill 0.4) (layers "F.Cu" "B.Cu") (net 43))
+  (segment (start 171.4425 76.7175) (end 173.05 78.325) (width 0.25) (layer "B.Cu") (net 43))
+  (segment (start 206.52 87.778356) (end 207.09125 87.207106) (width 0.25) (layer "B.Cu") (net 43))
+  (segment (start 201.570333 94.932523) (end 200.8 95.702856) (width 0.25) (layer "B.Cu") (net 43))
+  (segment (start 192.231454 93.168545) (end 193.4375 94.374591) (width 0.25) (layer "B.Cu") (net 43))
+  (segment (start 203.997477 92.500333) (end 203.857023 92.500333) (width 0.25) (layer "B.Cu") (net 43))
+  (segment (start 173.05 78.325) (end 173.05 79.25) (width 0.25) (layer "B.Cu") (net 43))
+  (segment (start 202.4 85.559644) (end 203.471606 86.63125) (width 0.25) (layer "B.Cu") (net 43))
+  (segment (start 207.2 96.29375) (end 207.2 95.702856) (width 0.25) (layer "B.Cu") (net 43))
+  (segment (start 207.09125 86.63125) (end 209.6625 86.63125) (width 0.25) (layer "B.Cu") (net 43))
+  (segment (start 171.4575 76.7175) (end 171.4425 76.7175) (width 0.25) (layer "B.Cu") (net 43))
+  (segment (start 201.570333 94.932523) (end 201.570333 92.500333) (width 0.25) (layer "B.Cu") (net 43))
+  (segment (start 200.8 95.702856) (end 200.8 96.29375) (width 0.25) (layer "B.Cu") (net 43))
+  (segment (start 198.3375 91.43125) (end 200.59022 91.43125) (width 0.25) (layer "B.Cu") (net 43))
+  (segment (start 191.9625 90.850394) (end 193.286053 92.173947) (width 0.25) (layer "B.Cu") (net 43))
+  (segment (start 203.997477 92.500333) (end 203.997477 91.512523) (width 0.25) (layer "B.Cu") (net 43))
+  (segment (start 202.4 84.96875) (end 202.4 85.559644) (width 0.25) (layer "B.Cu") (net 43))
+  (segment (start 193.4375 94.374591) (end 193.4375 95.39375) (width 0.25) (layer "B.Cu") (net 43))
+  (segment (start 174.125 74.05) (end 171.4575 76.7175) (width 0.25) (layer "B.Cu") (net 43))
+  (segment (start 200.59022 91.43125) (end 200.595735 91.425735) (width 0.25) (layer "B.Cu") (net 43))
+  (segment (start 207.12 86.66) (end 207.09125 86.63125) (width 0.25) (layer "B.Cu") (net 43))
+  (segment (start 203.109971 81.088204) (end 203.548844 80.649331) (width 0.25) (layer "B.Cu") (net 43))
+  (segment (start 191.9625 90.25) (end 191.9625 90.850394) (width 0.25) (layer "B.Cu") (net 43))
+  (segment (start 203.471606 86.63125) (end 207.09125 86.63125) (width 0.25) (layer "B.Cu") (net 43))
+  (segment (start 203.548844 80.649331) (end 203.548844 78.525481) (width 0.25) (layer "B.Cu") (net 43))
+  (segment (start 168.775 74.05) (end 171.4425 76.7175) (width 0.25) (layer "B.Cu") (net 43))
+  (segment (start 207.2 95.702856) (end 203.997477 92.500333) (width 0.25) (layer "B.Cu") (net 43))
+  (segment (start 203.548844 78.525481) (end 203.702529 78.371796) (width 0.25) (layer "B.Cu") (net 43))
+  (segment (start 207.09125 87.207106) (end 207.09125 86.63125) (width 0.25) (layer "B.Cu") (net 43))
+  (segment (start 203.997477 91.512523) (end 206.22 89.29) (width 0.25) (layer "B.Cu") (net 43))
+  (segment (start 201.570333 92.500333) (end 203.857023 92.500333) (width 0.25) (layer "B.Cu") (net 43))
   (zone (net 43) (net_name "GND") (layer "F.Cu") (hatch edge 0.508)
     (connect_pads (clearance 0.508))
